File: PSU_3V3.sch (KiCad schematic (older format))
At the start: 54 parts, among them J6 5V, J7 3V3, Q1 2N3906, U1 BD4830G, U10 LNK3202P, U11 AMS1117-3.3, U8 PC817, U9 TL431DBZ

Commit message: Minor fixes
Some typos
Fix test point outline
DRC/ERC pass
Parts:
- C18, C26: value 100µF -> 47µF
- MOV1: value MOV-10DxxxK -> MOV-10D420K
Other:
- note added: "Ultra-Fast\ntrr<=75ns (Imax < 63mA)\ntrr<=35ns (Imax < 80mA)"
- note removed: "Ultra-Fast\ntrr<=75ns"
Changed lines of the file:
@@
 encoding utf-8
 Sheet 2 2
-Title "3.3V 80mA power supply referenced to mains"
+Title "3.3V 60mA power supply referenced to mains"
 Date "2020-06-01"
 Rev "1.0"
@@
 P 6050 4500
 F 0 "C18" H 6168 4591 50  0000 L CNN
-F 1 "100µF" H 6168 4500 50  0000 L CNN
+F 1 "47µF" H 6168 4500 50  0000 L CNN
 F 2 "ValTronix:CP_Elec_6.3x7.7" H 6088 4350 50  0001 C CNN
 F 3 "~" H 6050 4500 50  0001 C CNN
@@
 	1    0    0    -1
 $EndComp
-Text Notes 4550 4300 3    50   ~ 0
-Ultra-Fast\ntrr<=75ns
+Text Notes 4550 3950 3    50   ~ 0
+Ultra-Fast\ntrr<=75ns (Imax < 63mA)\ntrr<=35ns (Imax < 80mA)
 Text Notes 5400 5050 1    50   ~ 0
 1.5mA
@@
 P 1700 4500
 F 0 "MOV1" H 1530 4553 59  0000 R CNN
-F 1 "MOV-10DxxxK" H 1530 4448 59  0000 R CNN
+F 1 "MOV-10D420K" H 1530 4448 59  0000 R CNN
 F 2 "ValTronix:RV_Disc_D12_W4.5_P7.5" H 1700 4500 50  0001 C CNN
 F 3 "https://www.bourns.com/docs/Product-Datasheets/MOV10D.pdf" H 1700 4500 50  0001 C CNN
@@
 P 6550 4500
 F 0 "C26" H 6668 4591 50  0000 L CNN
-F 1 "100µF" H 6668 4500 50  0000 L CNN
+F 1 "47µF" H 6668 4500 50  0000 L CNN
 F 2 "ValTronix:CP_Elec_6.3x7.7" H 6588 4350 50  0001 C CNN
 F 3 "~" H 6550 4500 50  0001 C CNN
@@
 Data
 89 50 4E 47 0D 0A 1A 0A 00 00 00 0D 49 48 44 52 00 00 00 B7 00 00 00 A0 08 02 00 00 00 C1 DF 6A
-EB 00 00 00 03 73 42 49 54 08 08 08 DB E1 4F E0 00 00 00 09 70 48 59 73 00 00 0D D7 00 00 0D D7
-01 42 28 9B 78 00 00 20 00 49 44 41 54 78 9C EC BD 79 80 A4 55 75 3E FC 9C BB BC 4B 55 F5 36 3D
+EB 00 00 00 03 73 42 49 54 08 08 08 DB E1 4F E0 00 00 00 09 70 48 59 73 00 00 0D AC 00 00 0D AC
+01 EF 06 C6 47 00 00 20 00 49 44 41 54 78 9C EC BD 79 80 A4 55 75 3E FC 9C BB BC 4B 55 F5 36 3D
 2B 0C 3B A2 80 4B 10 17 40 10 44 10 10 03 08 E2 8E B8 20 C6 18 8D 46 BF FC F4 A7 49 54 C4 0F 14
 70 10 10 04 24 83 03 24 D1 C8 22 B2 08 04 0D F2 21 42 64 0B 1A 14 18 F6 D9 E9 E9 A5 AA DE E5 DE

Commit message: Routage
Parts:
- removed C14: 6.8µF, ValTronix:CP_Radial_D10.0mm_P5.00mm, symbol Device:CP
- removed TP13: BP, Measurement_Points:Measurement_Point_Round-SMD-Pad_Small, symbol Connector:TestPoint
- removed TP15: FB, Measurement_Points:Measurement_Point_Round-SMD-Pad_Small, symbol Connector:TestPoint
- removed TP17: S, Measurement_Points:Measurement_Point_Round-TH_Big, symbol Connector:TestPoint
- added C16: 4.7µF, ValTronix:CP_Radial_D10.0mm_P5.00mm, symbol Device:CP
- added D5: SMBJ5.0A, ValTronix:D_SMB, symbol ValTronix:SMBJxxA
- added TP13: GNDA, Measurement_Points:Measurement_Point_Round-TH_Big, symbol Connector:TestPoint_Alt
- C17: renamed from C15; value 6.8µF -> 4.7µF; Part (none) -> ULD2G4R7MPD
- C18: renamed from C16; Part (none) -> CL31B104KBCNNNL
- C25: renamed from C22; footprint ValTronix:C_1206 -> ValTronix:C_0805
- C26: renamed from C17; footprint ValTronix:C_Disc_D5.1mm_W3.2mm_P5.00mm -> ValTronix:C_0805
- L1: value 2mH -> 1800µH; footprint ValTronix:L_Radial_D8.7mm_P5.00mm_Fastron_07HCP -> ValTronix:L_Bourns_SDR1006; Part (none) -> SDR1006-182KL
- L2: footprint ValTronix:L_Radial_D8.7mm_P5.00mm_Fastron_07HCP -> ValTronix:L_1210; Current 122mA -> 300mA; Part (none) -> LQH32CN100K23L
- NT1: renamed from R11; symbol Device:R -> Device:Net-Tie_2
- R28: renamed from R7; value 4.7k -> 33k
- RF1: footprint ValTronix:R_Axial_DIN0411_L9.9mm_D3.6mm_P5.08mm_Vertical -> ValTronix:R_Axial_DIN0414_L11.9mm_D4.5mm_P15.24mm_Horizontal
- SYM3: value 240V -> 230V
- TP1, TP10, TP16: footprint Measurement_Points:Measurement_Point_Square-TH_Small -> Measurement_Points:Measurement_Point_Square-SMD-Pad_Big
- TP11: value LRF -> L; footprint Measurement_Points:Measurement_Point_Round-SMD-Pad_Small -> Measurement_Points:Measurement_Point_Square-SMD-Pad_Small
- TP12: value D -> N; footprint Measurement_Points:Test_Point_Keystone_5019_Minature -> Measurement_Points:Measurement_Point_Round-TH_Big
- TP18: footprint Measurement_Points:Test_Point -> Measurement_Points:Measurement_Point_Round-TH_Big
- TP2: footprint Measurement_Points:Measurement_Point_Round-TH_Small -> Measurement_Points:Measurement_Point_Round-SMD-Pad_Small
- renumbered C18 to C19, C26 to C20, C19 to C21, C21 to C22, C20 to C24, D4 to D3, D3 to D4, FB3 to FB6, LD4 to LD3, R33 to R24, R26 to R25, R32 to R26, R34 to R27, R27 to R29, R28 to R30, R29 to R31, R30 to R32, R31 to R33, U8 to U11, U11 to U12, U1 to U13
Connections:
- net 3V3D: now also D4.3 (A), R24.1; no longer LD3.2 (A)
- net 5V: now also D5.1 (A1); no longer D4.3 (A), U11.1
- net D: no longer TP12.1
- net GNDA: now also TP13.1
- net GNDD: now also LD3.1 (K); no longer R24.2
- net L: now also TP11.1
- net LCC: now also C16.1
- net LRF: no longer TP11.1
- net N: now also TP12.1, C16.2, D5.2 (A2)
- net S+: now reaches C19.1, L1.2, L2.1, R26.1
- net S+: now also U11.1
- new net: LD3.2 (A), R24.2
Other:
- note added: "2.9V-3.6V garanteed"
- moved on the sheet: LD3, R24, R28
