File: EnergyMonitor.sch (KiCad schematic (older format))
At the start: 77 parts, among them J1 IN, J2 OUT, J3 V, J4 UART, J5 Conn_01x06, U12 MCP39F501, U13 74LVC1G14, U14 PC817, U2 MCP9700AT-ETT, U3 74LVC1G14, U4 74LVC1G14, U5 PC827, U6 PC817, U7 PC817, X1 SG-310, Y1 4MHz

Commit message: Minor fixes
Some typos
Fix test point outline
DRC/ERC pass
Parts:
- R1: value 330 -> 330k; Ref (none) -> MMU01020C3303FB300
- R2, R3: value 330 -> 330k
- SYM1: value 240V -> 230V
Other:
- note removed: "240V"
Changed lines of the file:
@@
 Wire Wire Line
 	3250 5050 3650 5050
-Text Notes 3450 6300 2    100  ~ 20
-240V
 $Comp
 L Graphic:SYM_Flash_Large SYM1
@@
 AR Path="/5DFE5F9E/5E3391D0" Ref="#SYM?"  Part="1"
 F 0 "SYM1" V 3100 5900 50  0001 C CNN
-F 1 "240V" V 3380 5900 50  0001 C CNN
+F 1 "230V" H 3369 5878 100 0000 L CNB
 F 2 "ValTronix:Symbol_HighVoltage_Silk" H 3240 5810 50  0001 C CNN
 F 3 "~" H 3650 5800 50  0001 C CNN
@@
 P 1300 4750
 F 0 "R3" H 1370 4841 50  0000 L CNN
-F 1 "330" H 1370 4750 50  0000 L CNN
+F 1 "330k" H 1370 4750 50  0000 L CNN
 F 2 "ValTronix:R_MELF_MMB-0207" V 1230 4750 50  0001 C CNN
 F 3 "~" H 1300 4750 50  0001 C CNN
@@
 P 1300 4400
 F 0 "R2" H 1370 4491 50  0000 L CNN
-F 1 "330" H 1370 4400 50  0000 L CNN
+F 1 "330k" H 1370 4400 50  0000 L CNN
 F 2 "ValTronix:R_MELF_MMB-0207" V 1230 4400 50  0001 C CNN
 F 3 "~" H 1300 4400 50  0001 C CNN
@@
 P 1300 4050
 F 0 "R1" H 1370 4141 50  0000 L CNN
-F 1 "330" H 1370 4050 50  0000 L CNN
+F 1 "330k" H 1370 4050 50  0000 L CNN
 F 2 "ValTronix:R_MELF_MMB-0207" V 1230 4050 50  0001 C CNN
 F 3 "~" H 1300 4050 50  0001 C CNN
 F 4 "0.1%" H 1370 3959 50  0000 L CNN "Préceision"
+F 5 "MMU01020C3303FB300" H 1300 4050 50  0001 C CNN "Ref"
 	1    1300 4050
 	1    0    0    -1
@@
 Data
 89 50 4E 47 0D 0A 1A 0A 00 00 00 0D 49 48 44 52 00 00 00 B7 00 00 00 A0 08 02 00 00 00 C1 DF 6A
-EB 00 00 00 03 73 42 49 54 08 08 08 DB E1 4F E0 00 00 00 09 70 48 59 73 00 00 0D D7 00 00 0D D7
-01 42 28 9B 78 00 00 20 00 49 44 41 54 78 9C EC BD 79 80 A4 55 75 3E FC 9C BB BC 4B 55 F5 36 3D
+EB 00 00 00 03 73 42 49 54 08 08 08 DB E1 4F E0 00 00 00 09 70 48 59 73 00 00 0D AC 00 00 0D AC
+01 EF 06 C6 47 00 00 20 00 49 44 41 54 78 9C EC BD 79 80 A4 55 75 3E FC 9C BB BC 4B 55 F5 36 3D
 2B 0C 3B A2 80 4B 10 17 40 10 44 10 10 03 08 E2 8E B8 20 C6 18 8D 46 BF FC F4 A7 49 54 C4 0F 14
 70 10 10 04 24 83 03 24 D1 C8 22 B2 08 04 0D F2 21 42 64 0B 1A 14 18 F6 D9 E9 E9 A5 AA DE E5 DE

Commit message: Routage
Parts:
- removed C25: 100nF, ValTronix:C_1206, symbol Device:C
- removed H3: L, Mounting_Holes:MountingHole_3.2mm_M3_ISO14580_Pad, symbol Mechanical:MountingHole_Pad
- removed J3: V, Wire_Pads:SolderWirePad_single_1-5mmDrill, symbol Connector:Screw_Terminal_01x01
- removed R21, R25: 10k, ValTronix:R_0805, symbol Device:R
- removed U13, U4: 74LVC1G14, ValTronix:SOT-353_SC-70-5, symbol ValTronix:74LVC1G14
- removed U14, U7: PC817, ValTronix:DIP-4_W7.62mm_LongPads, symbol ValTronix:PC817
- added C13: 100nF, ValTronix:C_0805, symbol Device:C
- added H3, H4: M2, Mounting_Holes:MountingHole_2.2mm_M2_ISO14580, symbol Mechanical:MountingHole
- added R12, R23: 1k, ValTronix:R_0805, symbol Device:R
- added TP15: GND, Measurement_Points:Measurement_Point_Round-TH_Big, symbol Connector:TestPoint
- added TP17: VCC, Measurement_Points:Measurement_Point_Square-SMD-Pad_Big, symbol Connector:TestPoint
- added U3, U4: H11L1SM, ValTronix:SMDIP-6_W9.53mm, symbol ValTronix:H11L1SM
- C14: renamed from C10; footprint ValTronix:C_1206 -> ValTronix:C_0805
- C15: renamed from C12; footprint ValTronix:C_1206 -> ValTronix:C_0805; Part (none) -> 08055C104KAT2A
- H1: renamed from H4; value N -> Nin
- H2: value Nload -> Nout
- H5: renamed from H1; value MountingHole -> M2; footprint Mounting_Holes:MountingHole_3.2mm_M3_ISO14580 -> Mounting_Holes:MountingHole_2.2mm_M2_ISO14580
- H6: renamed from H5; value MountingHole -> M2; footprint Mounting_Holes:MountingHole_3.2mm_M3_ISO14580 -> Mounting_Holes:MountingHole_2.2mm_M2_ISO14580
- JP1: footprint Wire_Connections_Bridges:WireConnection_1.00mmDrill -> Pin_Headers:Pin_Header_Straight_1x02_Pitch2.54mm
- R1: renamed from R9; footprint ValTronix:R_Shunt_8.75x5.6mm -> ValTronix:R_2512; symbol Device:R_Shunt -> Device:R
- R4: renamed from R1; footprint ValTronix:R_MELF_MMB-0207 -> ValTronix:R_MicroMELF_MMU-0102
- R5: renamed from R2; footprint ValTronix:R_MELF_MMB-0207 -> ValTronix:R_MicroMELF_MMU-0102
- R6: renamed from R3; footprint ValTronix:R_MELF_MMB-0207 -> ValTronix:R_MicroMELF_MMU-0102
- R7: renamed from R4; footprint ValTronix:R_0805 -> ValTronix:R_MicroMELF_MMU-0102
- U6: footprint ValTronix:DIP-4_W7.62mm_LongPads -> ValTronix:DIP-4_W7.62mm
- renumbered C24 to C10, C6 to C12, C3 to C2, C2 to C3, C7 to C6, C8 to C7, C9 to C8, C13 to C9, FB4 to FB3, FB5 to FB4, FB6 to FB5, LD2 to LD1, LD3 to LD2, LD1 to LD4, R12 to R10, R13 to R11, R23 to R13, R15 to R14, R16 to R15, R17 to R16, R18 to R17, R19 to R18, R22 to R19, R6 to R2, R14 to R20, R20 to R21, R24 to R22, R10 to R3, R5 to R8, R8 to R9, U12 to U1, U3 to U7
Connections:
- net +3V3: now also C13.2, R12.1, U3.6
- net GND: now also TP15.1, U3.2, U4.5
- net GNDD: now also C13.1, U3.5, U4.2
- net Nin: now also FB1.2
- net Nout: now also FB2.2, R1.2; no longer R1.4
- net RX_MON: now also R12.2, U3.4
- net TX: now also R23.1, U4.4
- net VCC: now also R23.2, TP17.1, U4.6
- net at R13.1: now also U4.1
- net at R22.2: now also U3.1
Other:
- moved on the sheet: C15, H5, H6, R13

Commit message: Première version produite
Parts:
- removed C13, C14, C15: 100nF, ValTronix:C_0805, symbol Device:C
- removed J4: UART, ValTronix:Pin_Header_Straight_1x04_Pitch2.54mm, symbol Connector_Generic:Conn_01x04
- removed LD1, LD2, LD4: LED_0805, ValTronix:LED_0805, symbol ValTronix:LED_0805
- removed R12, R13, R15, R17, R21, R22, R23: 1k, ValTronix:R_0805, symbol Device:R
- removed R14, R16: 2k, ValTronix:R_0805, symbol Device:R
- removed R18, R19: 10k, ValTronix:R_0805, symbol Device:R
- removed R20: 200, ValTronix:R_0805, symbol Device:R
- removed TP15: GND, Measurement_Points:Measurement_Point_Round-TH_Big, symbol Connector:TestPoint
- removed TP17: VCC, Measurement_Points:Measurement_Point_Square-SMD-Pad_Big, symbol Connector:TestPoint
- removed TP7: Test, Measurement_Points:Measurement_Point_Round-SMD-Pad_Small, symbol Connector:TestPoint_Probe
- removed U3, U4: H11L1SM, ValTronix:SMDIP-6_W9.53mm, symbol ValTronix:H11L1SM
- removed U5: PC827, ValTronix:DIP-8_W7.62mm, symbol Isolator:PC827
- removed U6: PC817, ValTronix:DIP-4_W7.62mm, symbol ValTronix:PC817
- removed U7: 74LVC1G14, ValTronix:SOT-353_SC-70-5, symbol ValTronix:74LVC1G14
- added FID1: Fiducial, Fiducials:Fiducial_0.5mm_Dia_1mm_Outer, symbol Mechanical:Fiducial
- added FID2, FID3, FID4, FID5: Fiducial, Fiducials:Fiducial_1mm_Dia_2mm_Outer, symbol Mechanical:Fiducial
- added H7, H8: M3, Mounting_Holes:MountingHole_3.2mm_M3_DIN965, symbol Mechanical:MountingHole
- added J4: UART, ValTronix:Pin_Header_Straight_1x06_Pitch2.54mm, symbol Connector_Generic:Conn_01x06
- added JP2: ~MCLR, ValTronix:JP3_SMD_12closed, symbol Jumper:SolderJumper_3_Bridged12
- H3, H4, H5, H6: value M2 -> M3; footprint Mounting_Holes:MountingHole_2.2mm_M2_ISO14580 -> Mounting_Holes:MountingHole_3.2mm_M3_DIN965
- J5: value Conn_01x06 -> IO
- X1: value SG-310 -> Q33310F70015812
Connections:
- net RX_MON is gone; now on net RX: U1.4 (RX)
- net TX_MON is gone; now on net TX: U1.12 (TX)
- net GND: now also J4.4 (Pin_4), J4.6 (Pin_6)
- net VCC: now also J4.1 (Pin_1)
- net ~MCLR: now also JP2.2 (C); no longer R10.2
- net ~RESET: now also JP2.3 (B)
- new net RXD: J4.3 (Pin_3)
- new net TXD: J4.2 (Pin_2)
- new net ~MCLR_PU: JP2.1 (A), R10.2
- new net ~RST: J4.5 (Pin_5)
Other:
- note added: "3.3V or 5V"
- note added: "<±25mA\nby DIO pin"
- note added: "All those connectors are NOT \nreferenced to mains"
- note added: "Caution:\n- No over/under voltage protection\n- No reverse polarity protection"
- note added: "Choose one option only!"
- note added: "Current measurement"
- note added: "GND guard"
- note added: "Isolated input/ouput pins"
- note added: "Master clock"
- note added: "PSU"
- note added: "Processing Unit"
- note added: "Temperature measurement"
- note added: "Voltage measurement"
- note removed: "1mA"
- note removed: "4800-8N1"
- moved on the sheet: C1, C10, C11, C12, C2, C3, C4, C5, C6, C7, C8, C9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
