File: InputOutput.sch (KiCad schematic (older format))
At the start: 53 parts, among them J6 5V, J7 3V3, Q1 2N3906, U10 LNK3202P, U11 PC817, U12 AMS1117-3.3, U13 BD4830G, U9 TL431DBZ

Commit message: Première version produite
Parts:
- removed C16, C17: 4.7µF, ValTronix:CP_Radial_D10.0mm_P5.00mm, symbol Device:CP
- removed C18: 0.1µF, ValTronix:C_1206, symbol Device:C
- removed C19, C20: 47µF, ValTronix:CP_Elec_6.3x7.7, symbol Device:CP
- removed C21, C23: 100nF, ValTronix:C_1206, symbol Device:C
- removed C22, C24: 10µF, ValTronix:CP_Elec_4x5.7, symbol Device:CP
- removed C25: 100nF, ValTronix:C_0805, symbol Device:C
- removed C26: 33nF, ValTronix:C_0805, symbol Device:C
- removed D1, D3: 1N4007, ValTronix:D_DO-41_SOD81_P10.16mm_Horizontal, symbol ValTronix:1N4007
- removed D2: UF4005, ValTronix:D_DO-41_SOD81_P10.16mm_Horizontal, symbol ValTronix:UF4005
- removed D4: FS0103MA, ValTronix:TO-92_Inline_Narrow_Oval, symbol ValTronix:FS01xxMA
- removed D5: SMBJ5.0A, ValTronix:D_SMB, symbol ValTronix:SMBJxxA
- removed DZ1: BZV55C3V9, ValTronix:D_MiniMELF, symbol ValTronix:BZV55Cxxx
- removed FB6: BLM18PG121SN1D, ValTronix:L_0805, symbol Device:Ferrite_Bead_Small
- removed J6: 5V, ValTronix:Pin_Header_Straight_1x02_Pitch2.54mm, symbol Connector_Generic:Conn_01x02
- removed J7: 3V3, ValTronix:Pin_Header_Straight_1x02_Pitch2.54mm, symbol Connector_Generic:Conn_01x02
- removed L1: 1800µH, ValTronix:L_Bourns_SDR1006, symbol Device:L_Core_Ferrite
- removed L2: 10µH, ValTronix:L_1210, symbol Device:L_Core_Ferrite
- removed LD3: LED_0805, ValTronix:LED_0805, symbol ValTronix:LED_0805
- removed MOV1: MOV-10D420K, ValTronix:RV_Disc_D12_W4.5_P7.5, symbol ValTronix:MOV-10DxxxK
- removed NT1: 0, ValTronix:R_0805, symbol Device:Net-Tie_2
- removed Q1: 2N3906, ValTronix:TO-92_Inline_Narrow_Oval, symbol ValTronix:2N3906
- removed R24, R31: 1k, ValTronix:R_0805, symbol Device:R
- removed R25: 100, ValTronix:R_Axial_DIN0414_L11.9mm_D4.5mm_P15.24mm_Horizontal, symbol ValTronix:RFP
- removed R26: 560, ValTronix:R_0805, symbol Device:R
- removed R27: 10, ValTronix:R_0805, symbol Device:R
- removed R28: 33k, ValTronix:R_0805, symbol Device:R
- removed R29: 12k, ValTronix:R_0805, symbol Device:R
- removed R30: 30k, ValTronix:R_0805, symbol Device:R
- removed R32, R33: 470, ValTronix:R_0805, symbol Device:R
- removed RF1: 8.2, ValTronix:R_Axial_DIN0414_L11.9mm_D4.5mm_P15.24mm_Horizontal, symbol ValTronix:RF
- removed SYM3: 230V, ValTronix:Symbol_HighVoltage_Silk, symbol Graphic:SYM_Flash_Large
- removed TP1: 5V, Measurement_Points:Measurement_Point_Square-SMD-Pad_Big, symbol Connector:TestPoint_Flag
- removed TP10: +3V3A, Measurement_Points:Measurement_Point_Square-SMD-Pad_Big, symbol Connector:TestPoint_Flag
- removed TP11: L, Measurement_Points:Measurement_Point_Square-SMD-Pad_Small, symbol Connector:TestPoint
- removed TP12: N, Measurement_Points:Measurement_Point_Round-TH_Big, symbol Connector:TestPoint
- removed TP13: GNDA, Measurement_Points:Measurement_Point_Round-TH_Big, symbol Connector:TestPoint_Alt
- removed TP14: Vz, Measurement_Points:Measurement_Point_Round-SMD-Pad_Small, symbol Connector:TestPoint
- removed TP16: +3V3D, Measurement_Points:Measurement_Point_Square-SMD-Pad_Big, symbol Connector:TestPoint_Flag
- removed TP18: GNDD, Measurement_Points:Measurement_Point_Round-TH_Big, symbol Connector:TestPoint_Alt
- removed TP19: Cr, Measurement_Points:Measurement_Point_Round-SMD-Pad_Small, symbol Connector:TestPoint_Probe
- removed TP2: ~RESET, Measurement_Points:Measurement_Point_Round-SMD-Pad_Small, symbol Connector:TestPoint
- removed U10: LNK3202P, ValTronix:PDIP-8C, symbol ValTronix:LNK3202P
- removed U11: PC817, ValTronix:DIP-4_W7.62mm_LongPads, symbol Isolator:PC817
- removed U12: AMS1117-3.3, ValTronix:SOT-223-3_TabPin2, symbol ValTronix:AMS1117-3.3
- removed U13: BD4830G, ValTronix:SSOP-5_2.9x2.8mm_Pitch0.95mm, symbol ValTronix:BD48xxG
- removed U9: TL431DBZ, ValTronix:SOT-23, symbol Reference_Voltage:TL431DBZ
- added C14, C30: 100nF, ValTronix:C_0805, symbol Device:C
- added C15, C28, C29: 100nF, ValTronix:C_0603, symbol Device:C
- added LD1, LD2, LD4: LED_0805, ValTronix:LED_0805, symbol ValTronix:LED_0805
- added R12, R36: 100k, ValTronix:R_0805, symbol Device:R
- added R13, R15, R16, R18, R20, R34: 1k, ValTronix:R_0805, symbol Device:R
- added R14, R35: 820, ValTronix:R_0805, symbol Device:R
- added R17, R19: 2k, ValTronix:R_0805, symbol Device:R
- added R21, R22: 10k, ValTronix:R_0805, symbol Device:R
- added R23: 200, ValTronix:R_0805, symbol Device:R
- added TP15: VCC, Measurement_Points:Measurement_Point_Square-SMD-Pad_Big, symbol Connector:TestPoint
- added TP7: GND, Measurement_Points:Measurement_Point_Round-TH_Big, symbol Connector:TestPoint
- added U14: 74LVC2G14, ValTronix:SOT-363_SC-70-6, symbol 74xGxx:74LVC2G14
- added U3, U5: 74LVC1G14, ValTronix:SOT-25, symbol ValTronix:74LVC1G14
- added U4, U6: H11L1SM, ValTronix:SMDIP-6_W9.53mm, symbol ValTronix:H11L1SM
- added U7, U8: PC827, ValTronix:SMDIP-8_W9.53mm, symbol Isolator:PC827
Connections:
- net +3V3: now also C28.1, C29.1, C30.1, R13.2, R21.1, U3.5 (VCC), U4.6, U5.5 (VCC)
- net GNDD: now also C28.2, C29.2, C30.2, LD1.1 (K), LD2.1 (K), LD4.1 (K), U3.3 (GND), U4.5, U5.3 (GND), U6.2, U7.2, U7.4, U8.5, U8.7
- net ~RESET: now also U8.8
- new net: R16.1, U5.4
- new net: R16.2, U6.1
- new net: R23.2, R34.2, U3.4
- new net: R21.2, R22.1
- new net: R14.1, U4.1
- new net: R14.2, U14.6
- new net: R35.1, U8.1
- new net: R35.2, U14.4
- new net D0_N: U7.7
- new net D0_P: U7.8
- new net D1_N: U7.5
- new net D1_P: U7.6
- new net D3_N: U8.4
- new net D3_P: U8.3
- new net DI3L: LD4.2 (A), R34.1
- new net DIO0: R17.1, R18.2
- new net DIO1: R19.1, R20.2
- new net DIO3: R23.1
- new net DO0: R17.2, U7.1
- new net DO0L: LD1.2 (A), R18.1
- new net DO1: R19.2, U7.3
- new net DO1L: LD2.2 (A), R20.1
- new net GND: C14.1, C15.1, TP7.1, U14.2 (GND), U14.2 (GND), U4.2, U6.5, U8.2
- new net RX: R13.1, U4.4
- new net RXD: U14.1
- new net TX: U5.2
- new net TXD: R15.1, U6.4
- new net VCC: C14.2, C15.2, R12.1, R15.2, R36.1, TP15.1, U14.5 (VCC), U14.5 (VCC), U6.6
- new net ~DI3: R22.2, U3.2, U8.6
- new net ~RST: R36.2, U14.3
- new net ~RXD: R12.2
Other:
- note added: "2mA"
- note added: "3.3V or 5V"
- note added: "4800-8N1"
- note added: "<50mA"
- note added: ">1.8mA\n<60mA"
- note added: "Caution:\n- No over/under voltage protection\n- No reverse polarity protection"
- note added: "Isolated inputs & outputs"
- note removed: "+3V3 analog (CAUTION: referenced to mains!)"
- note removed: "+3V3 digital (CAUTION: referenced to mains!)"
- note removed: "1.5mA"
- note removed: "2.9V-3.6V garanteed"
- note removed: "2V"
- note removed: "Crowbar and over voltage protection"
- note removed: "Ultra-Fast\ntrr<=75ns (Imax < 63mA)\ntrr<=35ns (Imax < 80mA)"
- note removed: "Voltage Supervisor"
- note removed: "minimum\nload: 3mA"
